Commit message: Changed structure to use only urdf/*.xacro

File: melfa/urdf/rv4fl.urdf.xacro (robot description, xacro)
@@ -5,8 +5,26 @@
     <color rgba="1.0 1.0 1.0 1.0"/>
   </material>
-  <xacro:include filename="$(find rovi_industrial)/melfa/urdf/rv4fl.xacro"/>
+  <xacro:include filename="$(find melfa_description)/urdf/rv4fl.xacro"/>
   <link name="base_link"/>
   <xacro:rv4fl parent="base_link">
     <origin xyz="0 0 0" rpy="0 0 0"/>
   </xacro:rv4fl>
+  <!-- ROS base_link to Robot Manufacturer World Coordinates transform -->
+  <link name="tool0" />
+  <joint name="link6-tool" type="fixed">
+    <origin xyz="0 0 0" rpy="0 0 0"/>
+    <parent link="link6"/>
+    <child link="tool0"/>
+  </joint>
+  <link name="base" />
+  <joint name="base_link-base" type="fixed">
+    <origin xyz="0 0 0" rpy="0 0 0"/>
+    <parent link="base_link"/>
+    <child link="base"/>
+  </joint>
+  <link name="world" />
+  <joint name="joint_w" type="fixed">
+    <parent link="world" />
+    <child link="base_link" />
+  </joint>
 </robot>

File: melfa/urdf/rv7fl.urdf.xacro (robot description, xacro)
@@ -10,3 +10,21 @@
     <origin xyz="0 0 0" rpy="0 0 0"/>
   </xacro:rv7fl>
+  <!-- ROS base_link to Robot Manufacturer World Coordinates transform -->
+  <link name="tool0" />
+  <joint name="link6-tool" type="fixed">
+    <origin xyz="0 0 0" rpy="0 0 0"/>
+    <parent link="link6"/>
+    <child link="tool0"/>
+  </joint>
+  <link name="base" />
+  <joint name="base_link-base" type="fixed">
+    <origin xyz="0 0 0" rpy="0 0 0"/>
+    <parent link="base_link"/>
+    <child link="base"/>
+  </joint>
+  <link name="world" />
+  <joint name="joint_w" type="fixed">
+    <parent link="world" />
+    <child link="base_link" />
+  </joint>
 </robot>
